File: LED_driver.brd (EAGLE design)
At the start: 40.1 x 30 mm, 17 parts

Commit message: New revision with MOSFET connected to the Enable of the IC
Parts:
- moved T2 14.3 mm to (10.4, 5.33), flipped to the top, turned to 0 degrees
- moved J1 1.78 mm to (17.8, 2.54)
- moved J8 1.27 mm to (12.7, 2.54)
Connections:
- removed net N$3: T2.1, U$3.LED-
- new net N$7: T2.2, U$1.3
- net 12V: now also T2.1; no longer U$1.3
- net LED-: now also U$3.LED-; no longer T2.2
Routing:
- net LED-: track 0.00 -> 10.7 mm, vias 2 -> 4
- net LED_PWM: track 4.09 -> 8.49 mm
- net N$7: track 0.00 -> 1.79 mm
- removed copper zone on layer 1, net N$3
- removed copper zone on layer 16, net N$3
Other:
- board size 40.1 x 30 mm -> 32.2 x 30 mm
Changed lines of the file:
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@@
 <grid distance="10" unitdist="mil" unit="mil" style="lines" multiple="1" display="no" altdistance="5" altunitdist="mil" altunit="mil"/>
 <layers>
-<layer number="1" name="Top" color="4" fill="1" visible="yes" active="yes"/>
+<layer number="1" name="Top" color="4" fill="1" visible="no" active="yes"/>
 <layer number="16" name="Bottom" color="1" fill="1" visible="yes" active="yes"/>
 <layer number="17" name="Pads" color="2" fill="1" visible="yes" active="yes"/>
@@
 <board>
 <plain>
-<wire x1="0" y1="0" x2="40.056" y2="0" width="0" layer="20"/>
-<wire x1="40.056" y1="0" x2="40.056" y2="29.962" width="0" layer="20"/>
-<wire x1="40.056" y1="29.962" x2="0" y2="29.962" width="0" layer="20"/>
+<wire x1="0" y1="0" x2="32.182" y2="0" width="0" layer="20"/>
+<wire x1="32.182" y1="0" x2="32.182" y2="29.962" width="0" layer="20"/>
+<wire x1="32.182" y1="29.962" x2="0" y2="29.962" width="0" layer="20"/>
 <wire x1="0" y1="29.962" x2="0" y2="0" width="0" layer="20"/>
 </plain>
@@
 <element name="C8" library="PowerComponents" package="CTAN(7.30_4.30MM)" value="47uF" x="5.588" y="10.668" rot="MR90"/>
 <element name="D1" library="BlueRobotics-Main" package="SMA" value="60V 3A" x="5.588" y="20.828" rot="R90"/>
-<element name="J1" library="SparkFun-Connectors" library_urn="urn:adsk.eagle:library:513" package="1X01" package3d_urn="urn:adsk.eagle:package:38028/1" value="" x="19.558" y="2.54"/>
-<element name="J8" library="SparkFun-Connectors" library_urn="urn:adsk.eagle:library:513" package="1X02_NO_SILK" package3d_urn="urn:adsk.eagle:package:38051/1" value="" x="13.97" y="2.54"/>
+<element name="J1" library="SparkFun-Connectors" library_urn="urn:adsk.eagle:library:513" package="1X01" package3d_urn="urn:adsk.eagle:package:38028/1" value="" x="17.78" y="2.54"/>
+<element name="J8" library="SparkFun-Connectors" library_urn="urn:adsk.eagle:library:513" package="1X02_NO_SILK" package3d_urn="urn:adsk.eagle:package:38051/1" value="" x="12.7" y="2.54"/>
 <element name="J9" library="SparkFun-Connectors" library_urn="urn:adsk.eagle:library:513" package="1X02_NO_SILK" package3d_urn="urn:adsk.eagle:package:38051/1" value="" x="7.62" y="2.54"/>
 <element name="R1" library="resistor" package="R2512" value="0.082 1W" x="16.002" y="6.35" rot="MR180"/>
 <element name="R2" library="resistor" package="R0603" value="140K" x="7.112" y="5.334"/>
 <element name="R7" library="resistor" package="R1206" value="NP" x="2.54" y="18.288" rot="R90"/>
-<element name="T2" library="zetex" package="SOT-23" value="" x="24.638" y="3.556" rot="MR270">
-<attribute name="MF" value="" x="24.638" y="3.556" size="1.778" layer="28" rot="MR270" display="off"/>
-<attribute name="MPN" value="" x="24.638" y="3.556" size="1.778" layer="28" rot="MR270" display="off"/>
-<attribute name="OC_FARNELL" value="unknown" x="24.638" y="3.556" size="1.778" layer="28" rot="MR270" display="off"/>
-<attribute name="OC_NEWARK" value="unknown" x="24.638" y="3.556" size="1.778" layer="28" rot="MR270" display="off"/>
+<element name="T2" library="zetex" package="SOT-23" value="" x="10.414" y="5.334">
+<attribute name="MF" value="" x="10.414" y="5.334" size="1.778" layer="27" display="off"/>
+<attribute name="MPN" value="" x="10.414" y="5.334" size="1.778" layer="27" display="off"/>
+<attribute name="OC_FARNELL" value="unknown" x="10.414" y="5.334" size="1.778" layer="27" display="off"/>
+<attribute name="OC_NEWARK" value="unknown" x="10.414" y="5.334" size="1.778" layer="27" display="off"/>
 </element>
 <element name="U$1" library="BlueRobotics-Main" package="SOIC8N-LJ" value="A6211" x="8.636" y="10.922"/>
@@
 <contactref element="C8" pad="+"/>
 <contactref element="C3" pad="1"/>
-<contactref element="U$1" pad="3"/>
 <contactref element="J9" pad="2"/>
 <contactref element="J9" pad="1"/>
 <polygon width="0.1524" layer="1">
-<vertex x="1.778" y="10.668"/>
-<vertex x="6.35" y="10.668"/>
-<vertex x="6.35" y="9.398"/>
+<vertex x="1.778" y="10.16"/>
+<vertex x="6.604" y="10.16"/>
+<vertex x="6.604" y="9.398"/>
 <vertex x="9.652" y="9.398"/>
 <vertex x="9.652" y="4.318"/>
-<vertex x="11.684" y="4.318"/>
-<vertex x="11.684" y="1.016"/>
+<vertex x="11.43" y="4.318"/>
+<vertex x="11.43" y="1.016"/>
 <vertex x="1.778" y="1.016"/>
 </polygon>
@@
 <vertex x="11.176" y="9.906"/>
 <vertex x="11.176" y="3.81"/>
-<vertex x="11.684" y="3.81"/>
-<vertex x="11.684" y="1.016"/>
+<vertex x="11.43" y="3.81"/>
+<vertex x="11.43" y="1.016"/>
 <vertex x="1.524" y="1.016"/>
 </polygon>
+<contactref element="T2" pad="1"/>
 </signal>
 <signal name="N$4">
@@
 <contactref element="R1" pad="2"/>
 <contactref element="U$1" pad="4"/>
-<contactref element="T2" pad="2"/>
 <polygon width="0.254" layer="16">
 <vertex x="24.384" y="3.556"/>
@@
 <vertex x="22.098" y="3.556"/>
 </polygon>
-<polygon width="0.254" layer="1">
-<vertex x="21.336" y="7.874"/>
-<vertex x="24.384" y="7.874"/>
-<vertex x="24.384" y="4.318"/>
-<vertex x="12.192" y="4.318"/>
-<vertex x="12.192" y="5.08"/>
-<vertex x="12.192" y="5.842"/>
-<vertex x="10.414" y="5.842"/>
-<vertex x="10.414" y="9.398"/>
-<vertex x="17.272" y="9.398"/>
-<vertex x="17.272" y="7.874"/>
-</polygon>
 <via x="20.828" y="6.604" extent="1-16" drill="0.35"/>
 <via x="21.844" y="5.334" extent="1-16" drill="0.35"/>
+<contactref element="U$3" pad="LED-"/>
+<polygon width="0.1524" layer="1">
+<vertex x="26.67" y="1.27"/>
+<vertex x="26.67" y="7.874"/>
+<vertex x="19.812" y="7.874"/>
+<vertex x="19.812" y="4.064"/>
+<vertex x="22.606" y="4.064"/>
+<vertex x="22.606" y="1.27"/>
+</polygon>
+<polygon width="0.254" layer="1">
+<vertex x="27.432" y="6.35"/>
+<vertex x="31.496" y="6.35"/>
+<vertex x="31.496" y="1.524"/>
+<vertex x="25.146" y="1.524"/>
+<vertex x="25.146" y="6.35"/>
+</polygon>
+<polygon width="0.254" layer="16">
+<vertex x="25.146" y="6.35"/>
+<vertex x="27.178" y="6.35"/>
+<vertex x="27.178" y="1.524"/>
+<vertex x="25.146" y="1.524"/>
+</polygon>
+<via x="25.908" y="5.334" extent="1-16" drill="0.35"/>
+<via x="26.162" y="2.286" extent="1-16" drill="0.35"/>
+<wire x1="10.546" y1="8.062" x2="10.546" y2="7.366" width="0.3048" layer="1"/>
+<wire x1="10.546" y1="7.366" x2="20.574" y2="7.366" width="0.3048" layer="1"/>
+<polygon width="0.1524" layer="16">
+<vertex x="23.876" y="7.62"/>
+<vertex x="25.654" y="7.62"/>
+<vertex x="25.654" y="1.524"/>
+<vertex x="23.876" y="1.524"/>
+</polygon>
 </signal>
 <signal name="VCC6211">
@@
 <contactref element="J1" pad="1"/>
 <contactref element="T2" pad="3"/>
-<wire x1="23.622" y1="2.5654" x2="19.558" y2="2.5654" width="0.254" layer="16"/>
-<wire x1="19.558" y1="2.5654" x2="19.558" y2="2.54" width="0.254" layer="16"/>
-</signal>
-<signal name="N$3">
-<contactref element="T2" pad="1"/>
-<contactref element="U$3" pad="LED-"/>
-<polygon width="0.254" layer="1">
-<vertex x="27.432" y="6.35"/>
-<vertex x="31.496" y="6.35"/>
-<vertex x="31.496" y="1.524"/>
-<vertex x="25.146" y="1.524"/>
-<vertex x="25.146" y="6.35"/>
-</polygon>
-<polygon width="0.254" layer="16">
-<vertex x="25.146" y="6.35"/>
-<vertex x="27.178" y="6.35"/>
-<vertex x="27.178" y="1.524"/>
-<vertex x="25.146" y="1.524"/>
-</polygon>
-<via x="25.908" y="5.334" extent="1-16" drill="0.35"/>
-<via x="26.162" y="2.286" extent="1-16" drill="0.35"/>
+<wire x1="17.78" y1="3.0734" x2="17.78" y2="2.54" width="0.254" layer="16"/>
+<wire x1="17.78" y1="2.54" x2="13.97" y2="6.35" width="0.3048" layer="1"/>
+<wire x1="13.97" y1="6.35" x2="11.4046" y2="6.35" width="0.3048" layer="1"/>
 </signal>
 <signal name="N$6">
@@
 </polygon>
 </signal>
+<signal name="N$7">
+<contactref element="T2" pad="2"/>
+<contactref element="U$1" pad="3"/>
+<wire x1="9.4742" y1="6.35" x2="9.276" y2="6.5482" width="0.3048" layer="1"/>
+<wire x1="9.276" y1="6.5482" x2="9.276" y2="8.062" width="0.3048" layer="1"/>
+</signal>
 </signals>

Commit message: continued revisions
Parts:
- added J2, J3, J4, J5: (no value), SparkFun-Connectors:1X01
- moved T2 11.8 mm to (22.1, 3.81), flipped to the bottom, turned to 270 degrees
- moved U$3 0.51 mm to (30.0, 7.11)
- moved C5 0.25 mm to (8.38, 16.5)
- moved D1 0.25 mm to (5.84, 20.8)
Connections:
- removed net N$7: T2.2, U$1.3
- new net N$3: J4.1, J5.1, T2.1, U$3.LED-
- net 12V: now also U$1.3; no longer T2.1
- net LED+: now also J2.1, J3.1
- net LED-: now also T2.2; no longer U$3.LED-
Routing:
- net LED_PWM: track 8.49 -> 3.42 mm
- net LED-: track 10.7 -> 8.22 mm, vias 4 -> 2
- net N$7: track 1.79 -> 0.00 mm
- net 12V: track 0.00 -> 1.51 mm
- added copper zone on layer 1, net N$3
- added copper zone on layer 16, net N$3
Other:
- board size 32.2 x 30 mm -> 32.7 x 25.1 mm
